Commit message: fixed wonky robot and image display

File: turtlebot3_description/urdf/_d435.gazebo.xacro (robot description, xacro)
@@ -19,5 +19,5 @@
       <!--<slip1>0</slip1>
       <slip2>0</slip2>-->
-      <kp>1e+13</kp>
+      <kp>1</kp>
       <kd>1</kd>
       <!--<max_vel>0.01</max_vel>
@@ -43,5 +43,4 @@
         <always_on>1</always_on>
         <update_rate>30</update_rate>
-        <visualize>1</visualize>
       </sensor>
       <sensor name="${camera_name}ired1" type="camera">

File: turtlebot3_description/urdf/_d435.urdf.xacro (robot description, xacro)
@@ -59,10 +59,4 @@
         </geometry>
       </collision>
-      <inertial>
-        <!-- The following are not reliable values, and should not be used for modeling -->
-        <mass value="0.564" />
-        <origin xyz="0 0 0" />
-        <inertia ixx="0.003881243" ixy="0.0" ixz="0.0" iyy="0.000498940" iyz="0.0" izz="0.003879257" />
-      </inertial>
     </link>
     <!-- camera depth joints and links -->

File: turtlebot3_description/urdf/turtlebot3_burger.urdf.xacro (robot description, xacro)
@@ -141,5 +141,5 @@
   </link>
   <joint name="camera_joint" type="fixed">
-    <origin xyz="0.064 -0.065 0.14" rpy="0 0 0"/>
+    <origin xyz="-0.032 0 0.20" rpy="0 0 0"/>
     <parent link="base_link"/>
     <child link="realsense_link"/>
@@ -149,14 +149,8 @@
      <origin xyz="0 0 0" rpy="1.57 0 1.57"/>
     </visual>
-    <collision>
-      <origin xyz="0.003 0.065 0.007" rpy="0 0 0"/>
-      <geometry>
-        <box size="0.012 0.132 0.020"/>
-      </geometry>
-    </collision>
   </link>
   <xacro:include filename="/home/carolina/turtle_ws/src/turtlebot3_description/urdf/_d435.urdf.xacro" />
   <xacro:sensor_d435 parent="realsense_link" name="d435" topics_ns="d435">
-    <origin xyz="-0.1 0 0" rpy="0 0 3.1456"/>
+    <origin xyz="0 0 0" rpy="0 0 0"/>
   </xacro:sensor_d435>
 </robot>
