Commit message: WORKING KEYPOINT POINTCLOUD

File: turtlebot3_description/urdf/_d435.urdf.xacro (robot description, xacro)
@@ -48,5 +48,5 @@
         <geometry>
           <!-- <box size="${d435_cam_width} ${d435_cam_height} ${d435_cam_depth}"/> -->
-          <mesh filename="package://realsense2_description/meshes/d435.dae" />
+          <mesh filename="/home/carolina/turtle_ws/src/realsense2_description/meshes/d435.dae" />
           <!--<mesh filename="package://realsense2_description/meshes/d435/d435.dae" />-->
         </geometry>

File: turtlebot3_description/urdf/turtlebot3_burger.urdf.xacro (robot description, xacro)
@@ -141,5 +141,5 @@
   </link>
   <joint name="camera_joint" type="fixed">
-    <origin xyz="-0.032 0 0.20" rpy="0 0 0"/>
+    <origin xyz="-0.05 0 0.18" rpy="0 0 0"/>
     <parent link="base_link"/>
     <child link="realsense_link"/>
